File: EAGLE/BPR-301 Circuit.sch (EAGLE design)
At the start: 0 parts

Commit message: adding files for sensors
Parts:
- added R1, R3, R5, R7: (no value), rcl:R-US_R0402
- added U$1, U$2: BPR-301, BPR-301:BPR-301
Connections:
- new net 3.3V: R1.2, R3.2, R5.2, R7.2
- new net GND: U$1.CATHODE, U$1.EMITTER, U$2.CATHODE, U$2.EMITTER
- new net N$1: R3.1, U$2.COLLECTOR
- new net N$2: R1.1, U$2.ANODE
- new net N$3: R5.1, U$1.COLLECTOR
- new net N$4: R7.1, U$1.ANODE
Other:
- note added: "Light Sensor"
