File: EAGLE/RecoveryBoard.sch (EAGLE design)
At the start: 78 parts, among them IC1 BD62120AEFJ-E2, J1 1725737, Q1 SI7617DN-T1-GE3, Q2 SI7617DN-T1-GE3, Q3 SIS412DN-T1-GE3, Q4 SIS412DN-T1-GE3, Q5 SI7617DN-T1-GE3, U1 STM32F042K6, U2 TPS54622RHLR, U3 BQ24616RGER

Commit message: handing off to dandrew
Parts:
- added C28: 2x 10uF, rcl:C-EUC0402
- added C29: 100uF, rcl:CPOL-US153CLV-0505
- added C30: 330uF, rcl:CPOL-US153CLV-0505
- added C31: 10uF, rcl:C-EUC0402
- added C32, C36: 0.1uF, rcl:C-EUC0402
- added C33: 1500pF, rcl:C-EUC0402
- added C34: 1.0uF, rcl:C-EUC0402
- added C35: 100uF, rcl:C-EUC0402
- added CM1: FTSH-105-XX-X-DV-K, J-Samtec-FTSH-105-XXX-DV-K-ARM-SWD:FTSH-105-XX-X-DV-K
- added L3: IHLP2020CZER220M11, IHLP2020CZER220M11:IHLP2020CZER220M11
- added R32: 2k, rcl:R-US_R0402
- added R33: 4.7, rcl:R-US_R0402
- added U4: TPS54356PWP, TPS54356PWP_TI:TPS54356PWP
- added U5: MBRS340T3G, MBRS340T3G:MBRS340T3G
- added Y1: ECS-160-10-36Q-ES-TR, ECS-160-10-36Q-ES-TR:ECS-160-10-36Q-ES-TR
- C10: value 10uF -> 0.1uF
- C3: value 4.7uF -> 20pF
- C4: value 0.01uF -> 20pF
- C5: value 0.1uF -> 3x 47uF
- C6: value 47pF -> 0.27nF
- C7: value 0.022uF -> 47nF
- C8: value optional -> 1uF
- C9: value 100uF -> 4.7uF
- L1: value SRP4030FA-3R3M -> IHLP2020CZER220M11; device SamacSys_Parts:SRP4030FA-3R3M -> IHLP2020CZER220M11:IHLP2020CZER220M11
- R1: value 35.7K -> 9.09k
- R2: value 8.06K -> 2k
- R3: value 100K -> 5.49k
- R4: value 3.74K -> 28k
- R5: value 10K -> 10k
- R6: value 2.21K -> 18.2k
- U2: value TPS54622RHLR -> XR76208EL-F; device TPS54622RHLR:TPS54622RHLR -> XR76208EL-F SPS:XR76208EL-F
Connections:
- net MOTOR+ renamed LAMOTOR+
- net MOTOR- renamed LAMOTOR-
- removed net 0: C10.1, C3.2, C4.2, C9.1, R2.1, R3.1, R6.1, U2.EPAD, U2.GND2, U2.GND3
- removed net 12V: C1.1, C2.1, IC1.VCC
- removed net 3.3V: C8.1, C9.2, L1.2, R10.2, R5.2, R7.2, R8.2, R9.2, U1.VDD, U1.VDDA, U1.VDDIO2
- removed net EN: U2.EN
- removed net N$3: R1.1, R2.2
- removed net SYSTEM2: C27.2, Q5.S_1, Q5.S_2, Q5.S_3, R31.1
- removed net TOBEDETERMINED: U1.PF0-OSC_IN, U1.PF1-OSC_OUT
- removed net VSNS: C8.2, R5.1, R6.2, U2.VSENSE
- new net +12V: C1.1, C2.1, C5.2, C6.2, IC1.VCC, J1.6, L1.2, R1.2
- new net +3V3: C30.+, C35.2, C36.2, CM1.VTREF, L3.1, R10.2, R7.2, R8.2, R9.2, U1.VDD, U1.VDDA, U1.VDDIO2, U4.VSENSE
- new net N$23: C9.2, U2.VCC
- new net N$25: L1.1, U2.SW_2, U2.SW_3, U2.SW_4, U2.SW_5
- new net N$26: C32.1, U4.BOOT
- new net N$27: C34.2, U4.VBIAS
- new net N$28: C33.2, R33.1
- new net N$29: C32.2, L3.2, R33.2, U4.PH, U4.PH_2, U5.-
- new net OSC_OUT: C4.1, U1.PF1-OSC_OUT, Y1.OUT/IN
- new net PVIN: C10.2, U2.VIN
- new net SW: C8.2, R3.1, U2.SW
- net GND: now also C10.1, C3.2, C30.-, C33.1, C34.1, C35.1, C36.1, C4.2, C5.1, C7.1, C9.1, CM1.GND, CM1.GND@2, CM1.GNDDET, J1.7, R2.1, R32.1, R4.1, U2.AGND, U2.AGND_2, U2.AGND_3, U4.AGND, U4.PGND, U4.PWRPAD, U5.+, Y1.GND
- net N$1: now also C3.1, U1.PF0-OSC_IN, Y1.IN/OUT; no longer R3.2, U2.RT/CLK
- net N$10: now also R5.2, U2.PGOOD; no longer C7.2, U2.SS/TR
- net N$11: now also C7.2, U2.SS; no longer C6.1, R4.2, U2.COMP
- net N$12: now also C6.1, R1.1, R2.2, U2.FB; no longer C4.1, R4.1
- net N$13: now also C8.1, U2.BST; no longer U2.PWRGD
- net N$4: now also C28.1, U2.PGND, U2.PGND_2, U2.PGND_3, U2.PGND_4, U2.PGND_5; no longer C3.1, R1.2, U2.VIN6
- net N$5: now also R32.2, R6.1, U2.EN/MODE; no longer C5.1, U2.BOOT
- net N$7: now also R3.2, U2.ILIM; no longer C5.2, L1.1, U2.PH, U2.PH_2
- net N$8: now also R4.2, U2.TON; no longer C6.2, C7.1
- net NRST: now also CM1.!RESET
- net SWCLK: now also CM1.SWDCLK/TCK
- net SWDIO: now also CM1.SWDIO/TMS
- net SYSTEM: now also C27.2, Q5.S_1, Q5.S_2, Q5.S_3, R31.1
- net VCC: now also R5.1
- net VIN: now also C28.2, C29.+, C31.1, R6.2, U2.PVIN, U2.PVIN_2, U2.PVIN_3, U2.PVIN_4, U2.PVIN_5, U2.PVIN_6, U2.PVIN_7, U2.PVIN_8, U4.VIN, U4.VIN_2; no longer C10.2, U2.PVIN4, U2.PVIN5
Other:
- note added: "12V SPS"
- note added: "3.3V SPS"
- note added: "DCM 12V"
- note added: "DCMGND"
- note added: "JTAG Connector"
- note added: "Needs to be set to 12V output"
- note added: "Terminals"
- note removed: "Need Motor and LA Terminal blocks"
- note removed: "Switching Power Supply 3.3V"
- note removed: "need 12 V supply"
- note removed: "this was in diagram?"
- moved on the sheet: C10, C3, C4, C5, C6, C7, C8, C9, R1, R2, R3, R4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

Commit message: implementing David's suggestions
Parts:
- removed L3: IHLP2020CZER220M11, IHLP2020CZER220M11:IHLP2020CZER220M11
- added L4: IHLP2020CZER220M11, IHLP2020CZER220M11:IHLP2020CZER220M11
- L1: value IHLP2020CZER220M11 -> IHLP2020CZER2R2M11; device IHLP2020CZER220M11:IHLP2020CZER220M11 -> IHLP2020CZER2R2M11:IHLP2020CZER2R2M11
- Q3: value SIS412DN-T1-GE3 -> SI7617DN-T1-GE3; device SamacSys_Parts:SIS412DN-T1-GE3 -> SamacSys_Parts:SI7617DN-T1-GE3
- Q5: value SI7617DN-T1-GE3 -> SIS412DN-T1-GE3; device SamacSys_Parts:SI7617DN-T1-GE3 -> SamacSys_Parts:SIS412DN-T1-GE3
- U2: DIS (none) -> Digikey; DPN (none) -> 1016-2078-ND
- U4: DIS (none) -> Digikey; DPN (none) -> 296-17073-ND
- U5: value MBRS340T3G -> D_MBRS340T3G; device MBRS340T3G:MBRS340T3G -> MBRS340T3G:D_MBRS340T3G
Connections:
- removed net ACDRV: R28.1
- removed net ACN: C17.2, U3.ACN
- removed net ANOTHER: C22.1, L2.1, Q3.S_1, Q3.S_2, Q3.S_3, Q4.D_1, Q4.D_2, Q4.D_3, Q4.D_4
- removed net SYSTEM1: Q3.D_1, Q3.D_2, Q3.D_3, Q3.D_4
- net +3V3: now also L4.1; no longer L3.1
- net ACP: now also Q1.D; no longer Q2.D_1, Q2.D_2, Q2.D_3, Q2.D_4
- net ADAPTER+: now also Q2.D; no longer Q1.D_1, Q1.D_2, Q1.D_3, Q1.D_4
- net GND: now also Q5.S; no longer Q4.S_1, Q4.S_2, Q4.S_3
- net HIDRV: now also Q4.G1; no longer Q3.G
- net LODRV: now also Q5.G1; no longer Q4.G
- net N$19: now also Q1.S, Q2.S; no longer Q1.S_1, Q1.S_2, Q1.S_3, Q2.S_1, Q2.S_2, Q2.S_3
- net N$20: now also Q1.G1, Q2.G1; no longer Q1.G, Q2.G
- net N$22: now also Q3.G1; no longer Q5.G
- net N$29: now also L4.2; no longer L3.2
- net PH: now also C22.1, L2.1, Q4.S, Q5.D
- net SYSTEM: now also C17.2, Q3.S, Q4.D, U3.ACN; no longer Q5.S_1, Q5.S_2, Q5.S_3
- net VBAT: now also Q3.D; no longer Q5.D_1, Q5.D_2, Q5.D_3, Q5.D_4
- net ~ACDRV: now also R28.1
Other:
- note added: "Adapter to System"
- note added: "BTST Cap"
- note added: "PackTherm"
- note added: "Status LEDs"
- note added: "VBAT"
- note added: "Voltage Dividers"
- note removed: "Section 1"
- note removed: "Section 2"
- note removed: "Section 3"
- note removed: "Section 4"
- note removed: "Section 5"
- note removed: "Section 6"
- moved on the sheet: C11, C14, CM1, L1, LED1, LED2, LED3, R19, R20, R21, R22, R23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

Commit message: Removed old schematics, and drastically simplified overall system. See design review notes from today.
Parts:
- removed C29: 100uF, rcl:CPOL-US153CLV-0505
- removed C30: 330uF, rcl:CPOL-US153CLV-0505
- removed C31: 10uF, rcl:C-EUC0402
- removed C32, C36: 0.1uF, rcl:C-EUC0402
- removed C33: 1500pF, rcl:C-EUC0402
- removed C34: 1.0uF, rcl:C-EUC0402
- removed C35: 100uF, rcl:C-EUC0402
- removed L4: IHLP2020CZER220M11, IHLP2020CZER220M11:IHLP2020CZER220M11
- removed R32: 2k, rcl:R-US_R0402
- removed R33: 4.7, rcl:R-US_R0402
- removed U2: XR76208EL-F, XR76208EL-F SPS:XR76208EL-F
- removed U4: TPS54356PWP, TPS54356PWP_TI:TPS54356PWP
- removed U5: D_MBRS340T3G, MBRS340T3G:D_MBRS340T3G
- added JP1, JP2: (no value), pinhead:PINHD-1X5
- added TP26, TP27, TP28, TP29, TP6: TEST-POINT, Tova:TEST-POINT
- added U10: TPS63070, ic-pwr-tps63070x:TPS63070X
- C10: value 0.1uF -> 10u; device rcl:C-EUC0402 -> oresat-rcl:C-EU0805-B-NOSILK
- C28: value 2x 10uF -> 22u; device rcl:C-EUC0402 -> oresat-rcl:C-EU0805-B-NOSILK
- C5: value 3x 47uF -> 10u; device rcl:C-EUC0402 -> oresat-rcl:C-EU0603-B-NOSILK; DIS (none) -> Digi-Key; DPN (none) -> 1276-1001-1-ND; MFR (none) -> Samsung; MPN (none) -> CL05B104KO5NNNC
- C6: value 0.27nF -> 10u; device rcl:C-EUC0402 -> oresat-rcl:C-EU0805-B-NOSILK
- C7: value 47nF -> 100n; device rcl:C-EUC0402 -> rcl_custom:C-EU0402-B-NOSILK; DIS (none) -> Digi-Key; DPN (none) -> 1276-1001-1-ND; MFR (none) -> Samsung; MPN (none) -> CL05B104KO5NNNC
- C8: value 1uF -> 22u; device rcl:C-EUC0402 -> oresat-rcl:C-EU0603-B-NOSILK; DIS (none) -> Digi-Key; DPN (none) -> 1276-1001-1-ND; MFR (none) -> Samsung; MPN (none) -> CL05B104KO5NNNC
- C9: value 4.7uF -> 22u; device rcl:C-EUC0402 -> oresat-rcl:C-EU0805-B-NOSILK
- L1: value IHLP2020CZER2R2M11 -> 1.5 uH; device IHLP2020CZER2R2M11:IHLP2020CZER2R2M11 -> L-Coilcraft-XFL4020:L-COILCRAFT-XFL4020; DIS (none) -> Mouser; DPN (none) -> 994-XFL4020-152MEB; MFR (none) -> Coilcraft; MPN (none) -> XFL4020-152ME
- R1: value 9.09k -> 10k; device rcl:R-US_R0402 -> rcl_custom:R-US_0402-B-NOSILK; DIS (none) -> Digi-Key; DPN (none) -> 1276-4275-1-ND; MFR (none) -> Samsung; MPN (none) -> RC1005F6653CS
- R2: value 2k -> 470k; device rcl:R-US_R0402 -> rcl_custom:R-US_0402-B-NOSILK; DIS (none) -> Digi-Key; DPN (none) -> 1276-4275-1-ND; MFR (none) -> Samsung; MPN (none) -> RC1005F6653CS
- R3: value 5.49k -> 100k; device rcl:R-US_R0402 -> rcl_custom:R-US_0402-B-NOSILK; DIS (none) -> Digi-Key; DPN (none) -> 1276-4275-1-ND; MFR (none) -> Samsung; MPN (none) -> RC1005F6653CS
- R4: value 28k -> 10k; device rcl:R-US_R0402 -> rcl_custom:R-US_0402-B-NOSILK; DIS (none) -> Digi-Key; DPN (none) -> 1276-4275-1-ND; MFR (none) -> Samsung; MPN (none) -> RC1005F6653CS
- R5: value 10k -> NP; device rcl:R-US_R0402 -> rcl_custom:R-US_0402-B-NOSILK; DIS (none) -> Digi-Key; DPN (none) -> 1276-4275-1-ND; MFR (none) -> Samsung; MPN (none) -> RC1005F6653CS
- R6: value 18.2k -> NP; device rcl:R-US_R0402 -> rcl_custom:R-US_0402-B-NOSILK; DIS (none) -> Digi-Key; DPN (none) -> 1276-4275-1-ND; MFR (none) -> Samsung; MPN (none) -> RC1005F6653CS
Connections:
- removed net +3V3: C30.+, C35.2, C36.2, CM1.VTREF, L4.1, R10.2, R7.2, R8.2, R9.2, U1.VDD, U1.VDDA, U1.VDDIO2, U4.VSENSE
- removed net N$10: R5.2, U2.PGOOD
- removed net N$11: C7.2, U2.SS
- removed net N$12: C6.1, R1.1, R2.2, U2.FB
- removed net N$13: C8.1, U2.BST
- removed net N$23: C9.2, U2.VCC
- removed net N$25: L1.1, U2.SW_2, U2.SW_3, U2.SW_4, U2.SW_5
- removed net N$26: C32.1, U4.BOOT
- removed net N$27: C34.2, U4.VBIAS
- removed net N$28: C33.2, R33.1
- removed net N$29: C32.2, L4.2, R33.2, U4.PH, U4.PH_2, U5.-
- removed net N$4: C28.1, U2.PGND, U2.PGND_2, U2.PGND_3, U2.PGND_4, U2.PGND_5
- removed net N$5: R32.2, R6.1, U2.EN/MODE
- removed net N$7: R3.2, U2.ILIM
- removed net N$8: R4.2, U2.TON
- removed net PVIN: C10.2, U2.VIN
- removed net SW: C8.2, R3.1, U2.SW
- removed net VIN: C28.2, C29.+, C31.1, R6.2, U2.PVIN, U2.PVIN_2, U2.PVIN_3, U2.PVIN_4, U2.PVIN_5, U2.PVIN_6, U2.PVIN_7, U2.PVIN_8, U4.VIN, U4.VIN_2
- new net 3.3V: C28.1, C8.1, C9.1, CM1.VTREF, R2.2, R5.2, R7.2, R8.2, R9.2, TP6.1, U1.VDD, U1.VDDA, U1.VDDIO2, U10.VOUT
- new net TPS-EN: R1.1, R6.2, TP29.1, U10.EN, U10.PS/SYNC
- new net TPS-FB: R2.1, R3.2, U10.FB
- new net TPS-FB2: TP27.1, U10.FB2
- new net TPS-L1: L1.1, U10.L1
- new net TPS-L2: L1.2, U10.L2
- new net TPS-PG: R5.1, TP26.1, U10.PG
- new net TPS-VAUX: C7.1, U10.VAUX
- new net TPS-VSEL: R4.2, TP28.1, U10.VSEL
- new net VBUS: C10.1, C5.1, C6.1, R1.2, U10.VIN
- net +12V: no longer C5.2, C6.2, L1.2, R1.2
- net GND: now also C10.2, C28.2, C5.2, C6.2, C7.2, C8.2, C9.2, R3.1, R6.1, U10.GND, U10.PGND; no longer C10.1, C30.-, C33.1, C34.1, C35.1, C36.1, C5.1, C7.1, C9.1, R2.1, R32.1, U2.AGND, U2.AGND_2, U2.AGND_3, U4.AGND, U4.PGND, U4.PWRPAD, U5.+
- net VCC: no longer R5.1
Other:
- note added: "0603"
- note added: "0805"
- note added: "12V "Active" brushless motor TSINY TS37GB60-BL3625"
- note added: "12V Linear Actuator with Position Output Actuonix P16-50-64-12-P"
- note added: "9 pulse/rot (YLW)"
- note added: "DIR (WHT)"
- note added: "GND (BLK)"
- note added: "MOTOR+"
- note added: "MOTOR-"
- note added: "POT out"
- note added: "POT+"
- note added: "POT-"
- note added: "PWM IN (BLU)"
- note added: "Power (12V - RED)"
- note removed: "12V SPS"
- note removed: "3.3V SPS"
- note removed: "Needs to be set to 12V output"

Commit message: 1-8-2020
Parts:
- removed U$1, U$2: BPR-301, BPR-301:BPR-301
- added SENSOR, SENSOR2: BPR-301, BPR-301:BPR-301
Connections:
- net GND: no longer U$1.CATHODE, U$1.EMITTER, U$2.CATHODE, U$2.EMITTER
- net N$14: no longer U$1.ANODE
- net N$2: no longer U$2.COLLECTOR
- net N$6: no longer U$2.ANODE
- net N$9: no longer U$1.COLLECTOR
Changed lines of the file:
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@@
 <?xml version="1.0" encoding="utf-8"?>
 <!DOCTYPE eagle SYSTEM "eagle.dtd">
-<eagle version="9.5.1">
+<eagle version="9.4.2">
 <drawing>
 <settings>
@@
 <part name="SUPPLY3" library="supply2" library_urn="urn:adsk.eagle:library:372" deviceset="GND" device=""/>
 <part name="SUPPLY4" library="supply2" library_urn="urn:adsk.eagle:library:372" deviceset="GND" device=""/>
-<part name="U$1" library="BPR-301" deviceset="BPR-301" device=""/>
-<part name="U$2" library="BPR-301" deviceset="BPR-301" device=""/>
 <part name="R7" library="rcl" library_urn="urn:adsk.eagle:library:334" deviceset="R-US_" device="R0402" package3d_urn="urn:adsk.eagle:package:23547/3" value="42"/>
 <part name="R8" library="rcl" library_urn="urn:adsk.eagle:library:334" deviceset="R-US_" device="R0402" package3d_urn="urn:adsk.eagle:package:23547/3" value="105"/>
@@
 </part>
 <part name="GND39" library="supply1" deviceset="GND" device=""/>
-<part name="VBUS1" library="oresat-supplies" deviceset="VBUS" device=""/>
+<part name="VUMB" library="oresat-supplies" deviceset="VBUS" device="" value="VUMB"/>
 <part name="SUPPLY31" library="SparkFun-PowerSymbols" library_urn="urn:adsk.eagle:library:530" deviceset="3.3V" device=""/>
 <part name="SUPPLY32" library="SparkFun-PowerSymbols" library_urn="urn:adsk.eagle:library:530" deviceset="3.3V" device=""/>
 <part name="SUPPLY33" library="SparkFun-PowerSymbols" library_urn="urn:adsk.eagle:library:530" deviceset="3.3V" device=""/>
 <part name="SUPPLY34" library="SparkFun-PowerSymbols" library_urn="urn:adsk.eagle:library:530" deviceset="3.3V" device=""/>
+<part name="SENSOR" library="BPR-301" deviceset="BPR-301" device=""/>
+<part name="SENSOR2" library="BPR-301" deviceset="BPR-301" device=""/>
 </parts>
 <sheets>
@@
 <attribute name="VALUE" x="78.74" y="219.71" size="1.778" layer="96"/>
 </instance>
-<instance part="VBUS1" gate="1" x="48.26" y="255.27" smashed="yes">
+<instance part="VUMB" gate="1" x="48.26" y="255.27" smashed="yes">
 <attribute name="VALUE" x="48.26" y="255.524" size="1.778" layer="96" align="bottom-center"/>
 </instance>
@@
 <wire x1="69.85" y1="250.19" x2="81.28" y2="250.19" width="0.1524" layer="91"/>
 <junction x="81.28" y="250.19"/>
-<pinref part="VBUS1" gate="1" pin="VBUS"/>
+<pinref part="VUMB" gate="1" pin="VBUS"/>
 </segment>
 </net>
@@
 <instance part="SUPPLY3" gate="GND" x="358.14" y="172.72" smashed="yes"/>
 <instance part="SUPPLY4" gate="GND" x="365.76" y="172.72" smashed="yes"/>
-<instance part="U$1" gate="G$1" x="81.28" y="127" smashed="yes"/>
-<instance part="U$2" gate="G$1" x="81.28" y="157.48" smashed="yes"/>
 <instance part="R7" gate="G$1" x="63.5" y="157.48" smashed="yes" rot="R180">
 <attribute name="NAME" x="67.31" y="155.9814" size="1.778" layer="95" rot="R180"/>
@@
 <instance part="SUPPLY34" gate="G$1" x="54.61" y="135.89" smashed="yes">
 <attribute name="VALUE" x="54.61" y="138.684" size="1.778" layer="96" align="bottom-center"/>
+</instance>
+<instance part="SENSOR" gate="BPR-301" x="99.06" y="166.37" smashed="yes">
+<attribute name="NAME" x="93.06" y="177.91" size="1.778" layer="95"/>
+<attribute name="VALUE" x="93.06" y="175.37" size="1.778" layer="96"/>
+</instance>
+<instance part="SENSOR2" gate="BPR-301" x="99.06" y="137.16" smashed="yes">
+<attribute name="NAME" x="93.06" y="148.7" size="1.778" layer="95"/>
+<attribute name="VALUE" x="93.06" y="146.16" size="1.778" layer="96"/>
 </instance>
 </instances>
@@
 </segment>
 <segment>
-<pinref part="U$2" gate="G$1" pin="EMITTER"/>
 <wire x1="121.92" y1="162.56" x2="152.4" y2="162.56" width="0.1524" layer="91"/>
 <wire x1="152.4" y1="162.56" x2="152.4" y2="157.48" width="0.1524" layer="91"/>
 <pinref part="SUPPLY5" gate="GND" pin="GND"/>
-<pinref part="U$1" gate="G$1" pin="EMITTER"/>
 <wire x1="152.4" y1="157.48" x2="152.4" y2="132.08" width="0.1524" layer="91"/>
 <wire x1="152.4" y1="132.08" x2="152.4" y2="127" width="0.1524" layer="91"/>
 <wire x1="152.4" y1="127" x2="152.4" y2="109.22" width="0.1524" layer="91"/>
 <junction x="152.4" y="132.08"/>
-<pinref part="U$1" gate="G$1" pin="CATHODE"/>
 <wire x1="121.92" y1="132.08" x2="152.4" y2="132.08" width="0.1524" layer="91"/>
 <wire x1="152.4" y1="127" x2="121.92" y2="127" width="0.1524" layer="91"/>
 <junction x="152.4" y="127"/>
-<pinref part="U$2" gate="G$1" pin="CATHODE"/>
 <wire x1="121.92" y1="157.48" x2="152.4" y2="157.48" width="0.1524" layer="91"/>
 <junction x="152.4" y="157.48"/>
@@
 <segment>
 <pinref part="R8" gate="G$1" pin="1"/>
-<pinref part="U$2" gate="G$1" pin="COLLECTOR"/>
 <wire x1="68.58" y1="162.56" x2="81.28" y2="162.56" width="0.1524" layer="91"/>
 </segment>
@@
 <net name="N$6" class="0">
 <segment>
-<pinref part="U$2" gate="G$1" pin="ANODE"/>
 <pinref part="R7" gate="G$1" pin="1"/>
 <wire x1="81.28" y1="157.48" x2="68.58" y2="157.48" width="0.1524" layer="91"/>
@@
 <net name="N$9" class="0">
 <segment>
-<pinref part="U$1" gate="G$1" pin="COLLECTOR"/>
 <pinref part="R9" gate="G$1" pin="1"/>
 <wire x1="81.28" y1="132.08" x2="68.58" y2="132.08" width="0.1524" layer="91"/>
@@
 <segment>
 <pinref part="R10" gate="G$1" pin="1"/>
-<pinref part="U$1" gate="G$1" pin="ANODE"/>
 <wire x1="68.58" y1="127" x2="81.28" y2="127" width="0.1524" layer="91"/>
 </segment>
