File: EAGLE/RecoveryBoard.sch (EAGLE design)
At the start: 88 parts, among them IC1 BD62120AEFJ-E2, Q6 MOSFET-PCH-SOT23-6, U1 STM32F042K6, U10 TPS63070, Y1 ECS-160-10-36Q-ES-TR

Commit message: beginning routing
Connections:
- net N$4 renamed DCM+
- net N$8 renamed PULSEOUT
- removed net N$1: LA.2
- new net N$30: C14.1, R20.1
- net GND: now also U$5.EP
- net LAMOTOR-: now also LA.2
Other:
- moved on the sheet: C14
Changed lines of the file:
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@@
 <attribute name="VALUE" x="190.246" y="157.099" size="1.016" layer="96"/>
 </instance>
-<instance part="C14" gate="CE" x="196.85" y="161.29" smashed="yes">
-<attribute name="NAME" x="197.866" y="161.925" size="1.016" layer="95"/>
-<attribute name="VALUE" x="197.866" y="157.099" size="1.016" layer="96"/>
+<instance part="C14" gate="CE" x="196.85" y="158.75" smashed="yes">
+<attribute name="NAME" x="197.866" y="159.385" size="1.016" layer="95"/>
+<attribute name="VALUE" x="197.866" y="154.559" size="1.016" layer="96"/>
 </instance>
 <instance part="R20" gate="R" x="196.85" y="167.64" smashed="yes" rot="R90">
@@
 <wire x1="148.59" y1="158.75" x2="166.37" y2="158.75" width="0.1524" layer="91"/>
 <junction x="166.37" y="158.75"/>
+<pinref part="U$5" gate="G$1" pin="EP"/>
+<wire x1="171.45" y1="161.29" x2="171.45" y2="157.48" width="0.1524" layer="91"/>
+<wire x1="171.45" y1="157.48" x2="166.37" y2="157.48" width="0.1524" layer="91"/>
+<wire x1="166.37" y1="157.48" x2="166.37" y2="158.75" width="0.1524" layer="91"/>
 </segment>
 <segment>
@@
 <pinref part="C14" gate="CE" pin="2"/>
 <pinref part="SUPPLY15" gate="GND" pin="GND"/>
-<wire x1="196.85" y1="156.21" x2="196.85" y2="152.4" width="0.1524" layer="91"/>
+<wire x1="196.85" y1="153.67" x2="196.85" y2="152.4" width="0.1524" layer="91"/>
 </segment>
 <segment>
@@
 <wire x1="148.59" y1="173.99" x2="114.3" y2="173.99" width="0.1524" layer="91"/>
 <junction x="114.3" y="173.99"/>
+</segment>
+</net>
+<net name="N$30" class="0">
+<segment>
+<pinref part="C14" gate="CE" pin="1"/>
+<pinref part="R20" gate="R" pin="1"/>
+<wire x1="196.85" y1="161.29" x2="196.85" y2="162.56" width="0.1524" layer="91"/>
 </segment>
 </net>
@@
 <wire x1="453.39" y1="294.64" x2="453.39" y2="289.56" width="0.1524" layer="91"/>
 <pinref part="SUPPLY38" gate="GND" pin="GND"/>
+<label x="455.93" y="294.64" size="1.778" layer="95"/>
 </segment>
 <segment>
@@
 <wire x1="427.99" y1="158.75" x2="427.99" y2="215.9" width="0.1524" layer="91"/>
 <wire x1="427.99" y1="215.9" x2="461.01" y2="215.9" width="0.1524" layer="91"/>
-</segment>
-</net>
-<net name="LAMOTOR-" class="0">
-<segment>
-<pinref part="IC1" gate="G$1" pin="OUT2"/>
-<wire x1="483.87" y1="161.29" x2="509.27" y2="161.29" width="0.1524" layer="91"/>
-<label x="509.27" y="161.29" size="1.6764" layer="95"/>
 </segment>
 </net>
@@
 </segment>
 </net>
-<net name="N$1" class="0">
+<net name="LAMOTOR-" class="0">
 <segment>
 <pinref part="LA" gate="A" pin="2"/>
 <wire x1="510.54" y1="161.29" x2="510.54" y2="213.36" width="0.1524" layer="91"/>
 <wire x1="510.54" y1="213.36" x2="461.01" y2="213.36" width="0.1524" layer="91"/>
+<pinref part="IC1" gate="G$1" pin="OUT2"/>
+<wire x1="483.87" y1="161.29" x2="510.54" y2="161.29" width="0.1524" layer="91"/>
+<label x="509.27" y="161.29" size="1.6764" layer="95"/>
 </segment>
 </net>
@@
 </segment>
 </net>
-<net name="N$4" class="0">
+<net name="DCM+" class="0">
 <segment>
 <pinref part="DCMOTOR" gate="A" pin="1"/>
@@
 <pinref part="Q6" gate="G$1" pin="D"/>
 <wire x1="426.72" y1="314.96" x2="426.72" y2="297.18" width="0.1524" layer="91"/>
+<label x="447.04" y="298.45" size="1.778" layer="95"/>
 </segment>
 </net>
@@
 </segment>
 </net>
-<net name="N$8" class="0">
+<net name="PULSEOUT" class="0">
 <segment>
 <pinref part="DCMOTOR" gate="A" pin="5"/>
 <wire x1="468.63" y1="287.02" x2="459.74" y2="287.02" width="0.1524" layer="91"/>
 <pinref part="R13" gate="G$1" pin="1"/>
-</segment>
-</net>
+<label x="454.66" y="287.02" size="1.778" layer="95"/>
+</segment>
+</net>

Commit message: Some fixes and polish.
Parts:
- renumbered DCMOTOR to J1, LA to J2
Connections:
- net N$15 renamed ARM-IN
- removed net N$23: C17.1, JP1.1, JP1.2, R15.2, R22.1, R25.2, U$5.BATT, U$8.S
- new net ARM-OUT: JP2.7, R25.1
- net VBAT: now also C17.1, JP1.1, JP1.2, R15.2, R22.1, R25.2, U$5.BATT, U$8.S; no longer JP2.7, R25.1
Other:
- note added: "12V power switch"
- note added: "Usually on"
Changed lines of the file:
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@@
 <part name="FRAME1" library="frames" library_urn="urn:adsk.eagle:library:229" deviceset="FRAME_B_L" device=""/>
 <part name="FRAME3" library="frames" library_urn="urn:adsk.eagle:library:229" deviceset="FRAME_C_L" device=""/>
-<part name="LA" library="pinhead" library_urn="urn:adsk.eagle:library:325" deviceset="PINHD-1X5" device="" package3d_urn="urn:adsk.eagle:package:22469/2"/>
-<part name="DCMOTOR" library="pinhead" library_urn="urn:adsk.eagle:library:325" deviceset="PINHD-1X5" device="" package3d_urn="urn:adsk.eagle:package:22469/2"/>
+<part name="J2" library="pinhead" library_urn="urn:adsk.eagle:library:325" deviceset="PINHD-1X5" device="" package3d_urn="urn:adsk.eagle:package:22469/2"/>
+<part name="J1" library="pinhead" library_urn="urn:adsk.eagle:library:325" deviceset="PINHD-1X5" device="" package3d_urn="urn:adsk.eagle:package:22469/2"/>
 <part name="C5" library="oresat-rcl" deviceset="C-EU" device="0603-B-NOSILK" value="10u">
 <attribute name="DIS" value="Digi-Key"/>
@@
 DISARM</text>
 <text x="40.64" y="203.2" size="1.778" layer="97">19V umbilical</text>
-<text x="212.09" y="257.81" size="1.778" layer="97">Do we still need an Arm input? there is no state where the board has power and is disarmed...this would free up a pin for a lock button</text>
+<text x="204.47" y="273.05" size="1.778" layer="97">Do we still need an Arm input? there is no state where the board has power and is disarmed...this would free up a pin for a lock button</text>
+<text x="292.1" y="251.46" size="1.778" layer="97">12V power switch</text>
+<text x="294.64" y="248.92" size="1.778" layer="97">Usually on</text>
 </plain>
 <instances>
@@
 </segment>
 </net>
-<net name="N$15" class="0">
+<net name="ARM-IN" class="0">
 <segment>
 <pinref part="JP2" gate="A" pin="6"/>
@@
 <wire x1="80.01" y1="246.38" x2="247.65" y2="246.38" width="0.1524" layer="91"/>
 <pinref part="R23" gate="R" pin="2"/>
-</segment>
-</net>
-<net name="VBAT" class="0">
+<label x="231.14" y="246.38" size="1.778" layer="95"/>
+</segment>
+</net>
+<net name="ARM-OUT" class="0">
 <segment>
 <pinref part="JP2" gate="A" pin="7"/>
@@
 <pinref part="R25" gate="R" pin="1"/>
 <wire x1="247.65" y1="236.22" x2="247.65" y2="242.57" width="0.1524" layer="91"/>
+<label x="231.14" y="242.57" size="1.778" layer="95"/>
 </segment>
 </net>
@@
 </segment>
 </net>
-<net name="N$23" class="0">
+<net name="VBAT" class="0">
 <segment>
 <pinref part="U$5" gate="G$1" pin="BATT"/>
@@
 <pinref part="R25" gate="R" pin="2"/>
 <wire x1="247.65" y1="201.93" x2="247.65" y2="226.06" width="0.1524" layer="91"/>
+<label x="259.08" y="201.93" size="1.778" layer="95"/>
 </segment>
 </net>
@@
 <attribute name="DRAWING_NAME" x="469.9" y="19.05" size="2.54" layer="94"/>
 </instance>
-<instance part="LA" gate="A" x="458.47" y="210.82" smashed="yes" rot="MR0">
+<instance part="J2" gate="A" x="458.47" y="210.82" smashed="yes" rot="MR0">
 <attribute name="NAME" x="464.82" y="219.075" size="1.778" layer="95" rot="MR0"/>
 <attribute name="VALUE" x="464.82" y="200.66" size="1.778" layer="96" rot="MR0"/>
 </instance>
-<instance part="DCMOTOR" gate="A" x="471.17" y="292.1" smashed="yes">
+<instance part="J1" gate="A" x="471.17" y="292.1" smashed="yes">
 <attribute name="NAME" x="464.82" y="300.355" size="1.778" layer="95"/>
 <attribute name="VALUE" x="464.82" y="281.94" size="1.778" layer="96"/>
@@
 </segment>
 <segment>
-<pinref part="DCMOTOR" gate="A" pin="2"/>
+<pinref part="J1" gate="A" pin="2"/>
 <wire x1="468.63" y1="294.64" x2="453.39" y2="294.64" width="0.1524" layer="91"/>
 <wire x1="453.39" y1="294.64" x2="453.39" y2="289.56" width="0.1524" layer="91"/>
@@
 </segment>
 <segment>
-<pinref part="LA" gate="A" pin="5"/>
+<pinref part="J2" gate="A" pin="5"/>
 <wire x1="461.01" y1="205.74" x2="476.25" y2="205.74" width="0.1524" layer="91"/>
 <pinref part="SUPPLY40" gate="GND" pin="GND"/>
@@
 <wire x1="453.39" y1="158.75" x2="427.99" y2="158.75" width="0.1524" layer="91"/>
 <label x="425.45" y="161.29" size="1.6764" layer="95"/>
-<pinref part="LA" gate="A" pin="1"/>
+<pinref part="J2" gate="A" pin="1"/>
 <wire x1="427.99" y1="158.75" x2="427.99" y2="215.9" width="0.1524" layer="91"/>
 <wire x1="427.99" y1="215.9" x2="461.01" y2="215.9" width="0.1524" layer="91"/>
@@
 <label x="302.26" y="187.96" size="1.27" layer="95"/>
 <wire x1="389.89" y1="259.08" x2="389.89" y2="292.1" width="0.1524" layer="91"/>
-<pinref part="DCMOTOR" gate="A" pin="3"/>
+<pinref part="J1" gate="A" pin="3"/>
 <wire x1="468.63" y1="292.1" x2="421.64" y2="292.1" width="0.1524" layer="91"/>
 <wire x1="421.64" y1="292.1" x2="389.89" y2="292.1" width="0.1524" layer="91"/>
@@
 </segment>
 <segment>
-<pinref part="LA" gate="A" pin="3"/>
+<pinref part="J2" gate="A" pin="3"/>
 <wire x1="461.01" y1="210.82" x2="491.49" y2="210.82" width="0.1524" layer="91"/>
 <wire x1="491.49" y1="210.82" x2="491.49" y2="220.98" width="0.1524" layer="91"/>
@@
 <net name="LAMOTOR-" class="0">
 <segment>
-<pinref part="LA" gate="A" pin="2"/>
+<pinref part="J2" gate="A" pin="2"/>
 <wire x1="510.54" y1="161.29" x2="510.54" y2="213.36" width="0.1524" layer="91"/>
 <wire x1="510.54" y1="213.36" x2="461.01" y2="213.36" width="0.1524" layer="91"/>
@@
 <net name="DCM_PWM" class="0">
 <segment>
-<pinref part="DCMOTOR" gate="A" pin="4"/>
+<pinref part="J1" gate="A" pin="4"/>
 <wire x1="468.63" y1="289.56" x2="429.26" y2="289.56" width="0.1524" layer="91"/>
 <wire x1="429.26" y1="289.56" x2="393.7" y2="289.56" width="0.1524" layer="91"/>
@@
 <net name="POT_OUT_AN" class="0">
 <segment>
-<pinref part="LA" gate="A" pin="4"/>
+<pinref part="J2" gate="A" pin="4"/>
 <wire x1="461.01" y1="208.28" x2="488.95" y2="208.28" width="0.1524" layer="91"/>
 <wire x1="488.95" y1="208.28" x2="488.95" y2="180.34" width="0.1524" layer="91"/>
@@
 <net name="DCM+" class="0">
 <segment>
-<pinref part="DCMOTOR" gate="A" pin="1"/>
+<pinref part="J1" gate="A" pin="1"/>
 <wire x1="426.72" y1="297.18" x2="468.63" y2="297.18" width="0.1524" layer="91"/>
 <pinref part="Q6" gate="G$1" pin="D"/>
@@
 <net name="PULSEOUT" class="0">
 <segment>
-<pinref part="DCMOTOR" gate="A" pin="5"/>
+<pinref part="J1" gate="A" pin="5"/>
 <wire x1="468.63" y1="287.02" x2="459.74" y2="287.02" width="0.1524" layer="91"/>
 <pinref part="R13" gate="G$1" pin="1"/>
