File: EAGLE/RecoveryBoard.brd (EAGLE design)
At the start: 120.9 x 50.8 mm, 84 parts, among them IC1 BD62120AEFJ-E2, Q6 MOSFET-PCH-SOT23-6, U1 STM32F042K6, U10 TPS63070, Y1 ECS-160-10-36Q-ES-TR

Commit message: starting grouping board components for layout
Parts:
- added C21: 10uF, oresat-rcl:.0805-C-NOSILK
- added D3: X-QE, D-Cree-XQE-LED:X-QE
- added R30: (no value), oresat-rcl:.0603-C-NOSILK
- added U$8: AO6405, Q--AO6405--P-CH MOSFET for Arm Switch:AO6405
- C12: value 4.7uF -> 10uF; device oresat-rcl:.0603-C-NOSILK -> oresat-rcl:.0805-C-NOSILK
- C14: value 2.2nF -> 0.1uF
- C15: device rcl:C0402 -> oresat-rcl:.0603-C-NOSILK
- C17: value 0.1uF -> 22uF
- R15: value 150K -> 2636
- R16: value 150K -> 1000
- R20: value 2.5K -> (none)
- U$3, U$4: value OPTOISOLATOR -> H11L1S(TA); device OptoIsolator:OPTOISOLATOR -> Q--H11L1S(TA)--OptoIsolator:H11L1S(TA)
- moved U$4 140.6 mm to (-4.80, -71.6)
- moved U$7 137.0 mm to (19.5, -54.4)
- moved R27 134.2 mm to (-8.51, -84.5)
- moved R29 134.1 mm to (14.2, -74.5)
- moved R26 130.4 mm to (-13.8, -75.5)
- moved R9 130.2 mm to (-44.7, -74.4)
- moved JP2 129.6 mm to (-94.2, -85.6), turned to 270 degrees
- moved U$3 129.3 mm to (-4.80, -61.2)
- moved R28 121.8 mm to (11.2, -64.5)
- moved R11 121.7 mm to (33.5, -56.4)
- moved R8 120.2 mm to (-44.6, -63.4)
- moved R36 118.9 mm to (25.8, -30.5)
- moved Q6 111.6 mm to (-63.3, -43.3)
- moved JP1 111.4 mm to (-94.1, -55.0), turned to 90 degrees
- moved R16 110.0 mm to (11.9, -33.2)
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Connections:
- removed net N$19 (its old number): C14.1, R20.1
- new net N$12: C21.1, R17.2, R18.2, R30.2, U$5.CELLS, U$5.VREF33
- new net N$23: C17.1, JP1.1, JP1.2, R15.2, R22.1, R25.2, U$5.BATT, U$8.S
- new net N$29: R29.1, U$4.GND
- net +12V: now also U$8.D1, U$8.D2, U$8.D3, U$8.D4
- net 3.3V: now also U$3.VCC, U$4.VCC; no longer U$3.P$3, U$4.P$3
- net ACOK: now also D3.CATHODE, U1.30
- net CHUTE: now also U$3.ANOD; no longer U$3.P$2
- net DROGUE: now also U$4.ANOD; no longer U$4.P$2
- net GND: now also C21.2
- net ISO-CHUTE: now also U$3.VO; no longer R28.1, U$3.P$4
- net ISO-DROGUE: now also U$4.VO; no longer R29.1, U$4.P$4
- net N$14: now also D3.ANODE, R30.1; no longer R17.2, R18.2, U$5.CELLS, U$5.VREF33
- net N$16: now also U$8.G
- net N$25: now also R28.1, U$3.GND; no longer C17.1, JP1.1, JP1.2, R15.2, R22.1, R25.2, U$5.BATT
- net N$26: now also U$4.CATH; no longer U$4.P$1
- net N$7: now also U$3.CATH; no longer U$3.P$1
Routing:
- added copper zone on layer 1, net GND

Commit message: beginning routing
Parts:
- moved SENSOR2 207.8 mm to (112.0, 44.5), turned to 270 degrees
- moved DCMOTOR 202.3 mm to (94.9, 4.33), turned to 180 degrees
- moved R9 194.9 mm to (106.7, 48.4), turned to 180 degrees
- moved R33 191.4 mm to (89.5, 23.5)
- moved LA 179.4 mm to (80.2, 4.33), turned to 0 degrees
- moved Q6 172.4 mm to (100.3, 10.8), turned to 180 degrees
- moved R34 166.9 mm to (94.1, 26.0), turned to 180 degrees
- moved U$2 165.9 mm to (98.9, 45.0)
- moved JP1 164.7 mm to (59.5, 4.33), turned to 180 degrees
- moved R25 153.5 mm to (44.0, 33.7), turned to 180 degrees
- moved C17 150.3 mm to (44.0, 36.3)
- moved JP2 150.1 mm to (20.2, 11.4)
- moved R6 149.4 mm to (36.1, 43.3), turned to 180 degrees
- moved C6 149.2 mm to (32.6, 29.1), turned to 270 degrees
- moved TP29 148.7 mm to (33.1, 43.2)
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Connections:
- net N$4 renamed DCM+
- net N$8 renamed PULSEOUT
- removed net N$1: LA.2
- new net N$30: C14.1, R20.1
- net GND: now also U$5.EP
- net LAMOTOR-: now also LA.2
Routing:
- net SENSOR1: track 0.00 -> 76.2 mm
- net VUMB: track 0.00 -> 65.2 mm, vias 0 -> 2
- net VBAT: track 0.00 -> 60.8 mm
- net PULSEOUT: track 0.00 -> 48.4 mm
- net 3.3V: track 0.00 -> 47.8 mm, vias 0 -> 3
- net N$15: track 0.00 -> 44.3 mm
- net POT_OUT_AN: track 0.00 -> 31.1 mm
- net +12V: track 0.00 -> 26.2 mm
- net TPS-EN: track 0.00 -> 25.5 mm
- net SENSOR_ON: track 0.00 -> 19.4 mm
- net N$6: track 0.00 -> 17.4 mm
- net LAMOTOR+: track 0.00 -> 17.4 mm
- net N$27: track 0.00 -> 13.6 mm
- net N$7: track 0.00 -> 13.4 mm
- net LAMOTOR-: track 0.00 -> 13.3 mm
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- added copper zone on layer 16, net 3.3V
Other:
- board size 120.9 x 50.8 mm -> 120.9 x 53.3 mm
- board text added: "BATT"
- board text added: "DCM+"
- board text added: "DCMOTOR"
- board text added: "LAMOTOR+"
- board text added: "LIN-ACT"
- board text added: "LiPo"
- board text added: "Recovery Board Rev1.0"
- board text added: "SPS"
- board text added: "this cap is too big"

Commit message: Some fixes and polish.
Parts:
- moved U$8 36.1 mm to (62.3, 9.60)
- moved R34 15.6 mm to (100.0, 11.5)
- moved Q6 1.74 mm to (100.0, 9.10), turned to 90 degrees
- renumbered DCMOTOR to J1, LA to J2
Connections:
- net N$15 renamed ARM-IN
- removed net N$23: C17.1, JP1.1, JP1.2, R15.2, R22.1, R25.2, U$5.BATT, U$8.S
- new net ARM-OUT: JP2.7, R25.1
- net VBAT: now also C17.1, JP1.1, JP1.2, R15.2, R22.1, R25.2, U$5.BATT, U$8.S; no longer JP2.7, R25.1
Routing:
- net SENSOR1: track 76.2 -> 0.00 mm
- net VUMB: track 65.2 -> 0.00 mm, vias 2 -> 0
- net VBAT: track 60.8 -> 0.00 mm
- net PULSEOUT: track 48.4 -> 0.00 mm
- net 3.3V: track 47.8 -> 0.00 mm, vias 3 -> 0
- net ARM-IN: track 44.3 -> 0.00 mm
- net POT_OUT_AN: track 31.1 -> 0.00 mm
- net TPS-EN: track 25.5 -> 0.00 mm
- net +12V: track 26.2 -> 2.02 mm
- net SENSOR_ON: track 19.4 -> 0.00 mm
- net LAMOTOR+: track 17.4 -> 0.00 mm
- net N$27: track 13.6 -> 0.00 mm
- net N$7: track 13.4 -> 0.00 mm
- net LAMOTOR-: track 13.3 -> 0.00 mm
- net OSC_OUT: track 12.9 -> 0.00 mm
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- added copper zone on layer 1, net DCM+
- added copper zone on layer 16, net GND
- removed copper zone on layer 16, net 3.3V
Other:
- board size 120.9 x 53.3 mm -> 120.9 x 54.6 mm
- board text added: "M+"
- board text added: "M-"
- board text added: "POT"
- board text added: "POT+"
- board text added: "POT-"
- board text removed: "DCM+"
