File: LV3.1/RecoveryBoard/eagle/RecoveryBoard.brd (EAGLE design)
At the start: 120.9 x 54.6 mm, 92 parts, among them IC1 BD62120AEFJ-E2, Q1 BSS123, Q2 BSS123, Q3 BSS123, Q6 MOSFET-PCH-SOT23-6, U1 STM32F042K6, U10 TPS63070, Y1 ECS-160-10-36Q-ES-TR

Commit message: adding libraries to repo and notes from design review
Parts:
- C15: value 0.1uF -> 100nF
- R15: value 2636 -> 26.36K
- R16: value 1000 -> 10K
Connections:
- removed net N$8: IC1.8, J2.2
- new net LAMOTOR+: IC1.2, J2.1
- net GND: now also IC1.7
- net LAMOTOR-: now also IC1.8, J2.2; no longer IC1.2, J2.1
Routing:
- net VBAT: track 91.5 -> 92.9 mm
- net N$28: track 14.8 -> 15.7 mm
Changed lines of the file:
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@@
 <attribute name="VALUE" x="78.035" y="34.555" size="0.4064" layer="27" rot="R180"/>
 </element>
-<element name="R15" library="oresat-rcl" package=".0603-C-NOSILK" value="2636" x="88.79" y="45.13" smashed="yes" rot="R180">
+<element name="R15" library="oresat-rcl" package=".0603-C-NOSILK" value="26.36K" x="88.79" y="45.13" smashed="yes" rot="R180">
 <attribute name="DIS" value="Digi-Key" x="54.5" y="109.9" size="1.778" layer="27" rot="R180" display="off"/>
 <attribute name="DPN" value="1276-4275-1-ND" x="54.5" y="109.9" size="1.778" layer="27" rot="R180" display="off"/>
@@
 <attribute name="VALUE" x="89.79" y="47.18" size="0.4064" layer="27" font="vector" ratio="15" rot="R180"/>
 </element>
-<element name="R16" library="oresat-rcl" package=".0603-C-NOSILK" value="1000" x="91.2" y="45.13" smashed="yes" rot="R180">
+<element name="R16" library="oresat-rcl" package=".0603-C-NOSILK" value="10K" x="91.2" y="45.13" smashed="yes" rot="R180">
 <attribute name="DIS" value="Digi-Key" x="53.1" y="109.9" size="1.778" layer="27" rot="R180" display="off"/>
 <attribute name="DPN" value="1276-4275-1-ND" x="53.1" y="109.9" size="1.778" layer="27" rot="R180" display="off"/>
@@
 </element>
 <element name="U$8" library="Q--Si7465DP--Vishay Power MOSFET with multple S+D leads" package="SI7465DP" value="SI7465DP" x="56.9" y="9.4" smashed="yes" rot="R90"/>
-<element name="C15" library="oresat-rcl" package=".0603-C-NOSILK" value="0.1uF" x="62.7" y="34.3" smashed="yes">
+<element name="C15" library="oresat-rcl" package=".0603-C-NOSILK" value="100nF" x="62.7" y="34.3" smashed="yes">
 <attribute name="NAME" x="63.1" y="33.7" size="0.4064" layer="25" font="vector" ratio="15" rot="R180"/>
 <attribute name="NAME" x="62.7" y="34.3" size="0.3" layer="33" ratio="15" align="center"/>
@@
 <attribute name="MOUSER_PART_NUMBER" value="755-BD62120AEFJ-E2" x="-12.2" y="-28.2" size="1.778" layer="27" display="off"/>
 <attribute name="MOUSER_PRICE-STOCK" value="https://www.mouser.com/Search/Refine.aspx?Keyword=755-BD62120AEFJ-E2" x="-12.2" y="-28.2" size="1.778" layer="27" display="off"/>
-<attribute name="NAME" x="-12.2" y="-28.2" size="1.27" layer="25" align="center"/>
+<attribute name="NAME" x="-12.3" y="-24.1" size="1.27" layer="25" align="center"/>
 <attribute name="VALUE" x="-12.2" y="-28.2" size="1.27" layer="27" align="center"/>
 </element>
@@
 <contactref element="IC1" pad="9"/>
 <contactref element="IC1" pad="1"/>
+<contactref element="IC1" pad="7"/>
 <wire x1="102.8" y1="43.2" x2="101.85" y2="43.6" width="0" layer="19" extent="1-1"/>
 <wire x1="105.97" y1="40.53" x2="102.8" y2="43.2" width="0" layer="19" extent="1-1"/>
@@
 <wire x1="23.8" y1="11.5" x2="24.4" y2="19.3" width="0" layer="19" extent="1-1"/>
 <wire x1="20.25" y1="11.37" x2="23.8" y2="11.5" width="0" layer="19" extent="1-1"/>
-<wire x1="-12.2" y1="-28.2" x2="20.25" y2="11.37" width="0" layer="19" extent="1-1"/>
+<wire x1="-9.488" y1="-27.565" x2="20.25" y2="11.37" width="0" layer="19" extent="1-1"/>
+<wire x1="-12.2" y1="-28.2" x2="-9.488" y2="-27.565" width="0" layer="19" extent="1-1"/>
 <wire x1="-14.912" y1="-30.105" x2="-12.2" y2="-28.2" width="0" layer="19" extent="1-1"/>
 <wire x1="-14.912" y1="-26.295" x2="-12.2" y2="-28.2" width="0" layer="19" extent="1-1"/>
@@
 <wire x1="80.55" y1="40.3" x2="80.35" y2="40.1" width="0.2" layer="1"/>
 </signal>
-<signal name="LAMOTOR-">
+<signal name="LAMOTOR+">
 <contactref element="IC1" pad="2"/>
 <contactref element="J2" pad="1"/>
@@
 <contactref element="R22" pad="2"/>
 <contactref element="U$5" pad="CSP"/>
-<wire x1="60.29" y1="28.27" x2="60.29" y2="29.81" width="0.2" layer="1"/>
-<wire x1="58.48" y1="31.62" x2="58.48" y2="33.21" width="0.2" layer="1"/>
-<wire x1="60.29" y1="29.81" x2="58.48" y2="31.62" width="0.2" layer="1"/>
-<wire x1="66.4" y1="32.78" x2="66.4" y2="30.88" width="0.2" layer="1"/>
-<wire x1="66.4" y1="30.88" x2="63.79" y2="28.27" width="0.2" layer="1"/>
-<wire x1="63.79" y1="28.27" x2="60.29" y2="28.27" width="0.2" layer="1"/>
+<wire x1="60.29" y1="28.27" x2="60.29" y2="28.81" width="0.2" layer="1"/>
+<wire x1="66.4" y1="32.78" x2="66.4" y2="30.88" width="1" layer="1"/>
+<wire x1="66.4" y1="30.88" x2="63.79" y2="28.27" width="1" layer="1"/>
+<wire x1="63.79" y1="28.27" x2="60.29" y2="28.27" width="1" layer="1"/>
+<wire x1="58.48" y1="33.21" x2="58.48" y2="30.32" width="0.1524" layer="1"/>
+<wire x1="58.48" y1="30.32" x2="59.2" y2="29.6" width="0.1524" layer="1"/>
+<wire x1="59.2" y1="29.6" x2="59.2" y2="28.7" width="0.1524" layer="1"/>
+<wire x1="59.2" y1="28.7" x2="59.63" y2="28.27" width="0.1524" layer="1"/>
+<wire x1="59.63" y1="28.27" x2="60.29" y2="28.27" width="0.1524" layer="1"/>
 </signal>
 <signal name="VBAT">
@@
 <contactref element="JP1" pad="1"/>
 <contactref element="R25" pad="2"/>
-<wire x1="57.83" y1="33.21" x2="57.83" y2="28.61" width="0.5" layer="1"/>
-<wire x1="57.83" y1="28.61" x2="57.49" y2="28.27" width="0.5" layer="1"/>
+<wire x1="57.63" y1="28.41" x2="57.49" y2="28.27" width="0.5" layer="1"/>
 <wire x1="57.49" y1="28.27" x2="57.49" y2="22.71" width="0.5" layer="1"/>
 <wire x1="57.49" y1="22.71" x2="63.5" y2="16.7" width="0.5" layer="1"/>
@@
 <wire x1="76.3" y1="29.5" x2="63.5" y2="16.7" width="0.5" layer="1"/>
 <wire x1="76.3" y1="41.4" x2="76.3" y2="29.5" width="0.5" layer="1"/>
+<wire x1="57.83" y1="33.21" x2="57.83" y2="30.37" width="0.1524" layer="1"/>
+<wire x1="57.83" y1="30.37" x2="58.7" y2="29.5" width="0.1524" layer="1"/>
+<wire x1="58.7" y1="29.5" x2="58.7" y2="28.6" width="0.1524" layer="1"/>
+<wire x1="58.7" y1="28.6" x2="58.4" y2="28.3" width="0.1524" layer="1"/>
+<wire x1="58.4" y1="28.3" x2="57.74" y2="28.3" width="0.1524" layer="1"/>
+<wire x1="57.74" y1="28.3" x2="57.63" y2="28.41" width="0.1524" layer="1"/>
+<wire x1="60.71" y1="9.4" x2="65.7" y2="11.2" width="0" layer="19" extent="1-1"/>
+<wire x1="59.44" y1="9.4" x2="60.71" y2="9.4" width="0" layer="19" extent="1-1"/>
+<wire x1="58.17" y1="9.4" x2="59.44" y2="9.4" width="0" layer="19" extent="1-1"/>
+<wire x1="60.79" y1="4.325" x2="60.71" y2="9.4" width="0" layer="19" extent="1-1"/>
+<wire x1="63.33" y1="4.325" x2="60.79" y2="4.325" width="0" layer="19" extent="1-1"/>
 </signal>
 <signal name="N$22">
@@
 <wire x1="91.7224" y1="24.2224" x2="91.7224" y2="22.5" width="0.2" layer="1"/>
 </signal>
-<signal name="N$8">
+<signal name="LAMOTOR-">
 <contactref element="J2" pad="2"/>
 <contactref element="IC1" pad="8"/>

Commit message: implementing design changes from 1/21/2020
Parts:
- removed SENSOR, SENSOR2: BPR-301, BPR-301:BPR-301
- added JP3: (no value), pinhead:1X03
- added Q4, Q5: BPR-301, Q--BPR-301--Phototransistor:BPR-301
- added TP1, TP2, TP3, TP4: TEST-POINT, Tova:2MM-TEST-POINT
- C1, C14: value 0.1uF -> 100n
- C11, C12, C21: value 10uF -> 10u
- C13: value 0.1uF -> 0.1u
- C15: value 100nF -> 100n
- C16: value 2.2nF -> 2.2n
- C17: value 22uF -> 22u
- C22: value 100uF -> 100n
- C3, C4: value 20pF -> 20p
- R27: value TBD -> 50
- moved IC1 105.1 mm to (86.9, 6.90), turned to 270 degrees
- moved D2 4.39 mm to (70.0, 33.4), turned to 90 degrees
- moved C15 3.80 mm to (62.6, 30.5)
- moved C13 1.24 mm to (62.4, 34.8)
- moved L2 0.73 mm to (65.7, 34.2)
Connections:
- net 3.3V: now also Q4.AN, Q4.C, Q5.AN, Q5.C; no longer SENSOR.AN, SENSOR.COLL, SENSOR2.AN, SENSOR2.COLL
- net CAN_RX: now also TP1.1
- net CAN_TX: now also TP2.1
- net GND: now also JP3.3
- net N$2: now also Q4.CAT; no longer SENSOR.CAT
- net N$5: now also Q5.CAT; no longer SENSOR2.CAT
- net SENSOR1: now also Q4.E; no longer SENSOR.EMIT
- net SENSOR2: now also Q5.E; no longer SENSOR2.EMIT
- net USART2_RX: now also JP3.1, TP3.1
- net USART2_TX: now also JP3.2, TP4.1
Routing:
- net USART2_RX: track 0.00 -> 34.9 mm, vias 0 -> 2
- net CAN_RX: track 0.00 -> 19.3 mm, vias 0 -> 2
- net USART2_TX: track 0.00 -> 17.4 mm, vias 0 -> 2
- net CAN_TX: track 0.00 -> 14.5 mm, vias 0 -> 2
- net LAMOTOR+: track 0.00 -> 13.2 mm
- net LAMOTOR-: track 0.00 -> 12.0 mm
- net VUMB: track 69.6 -> 80.4 mm, vias 1 -> 3
- net GND: track 8.96 -> 16.0 mm, vias 42 -> 91
- net 3.3V: track 317.8 -> 312.0 mm
- net DCM_PWM: track 34.5 -> 38.7 mm
- net DCMDIR: track 33.7 -> 37.2 mm
- net N$10: track 13.3 -> 10.0 mm
- net ISO-DROGUE: track 63.0 -> 65.7 mm
- net IN2: track 46.6 -> 49.1 mm
- net IN1: track 42.5 -> 44.9 mm
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Other:
- board text added: "TODO 1. I have CAN and USART Pins currenlty doing nothing 2. Need to add locking button"
- board text removed: "TODO 1. I have CAN and USART Pins currenlty doing nothing 2. Need to add locking button 3. Update H-Bridge symbol"

Commit message: created BOM
Parts:
- C17: value 22u -> 22uF
- R13: value 1.7K -> 1.69K
- R15: value 26.36K -> 26.4K
- R26, R27: value 50 -> 51.1
- R28: value 50 -> 10K
- R8, R9: value 439 -> 442
Routing:
- net N$28: track 15.6 -> 15.1 mm
Other:
- board text added: "GND"
- board text added: "USART2"
- board text added: "VBAT"
Changed lines of the file:
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@@
 <drawing>
 <settings>
-<setting alwaysvectorfont="no"/>
+<setting alwaysvectorfont="yes"/>
 <setting verticaltext="up"/>
 </settings>
@@
 2. Need to add locking button
 </text>
+<text x="75.9" y="15.5" size="1" layer="21" font="vector" ratio="20">USART2</text>
+<text x="60.9" y="1.35" size="0.635" layer="21" font="vector" ratio="20">VBAT</text>
+<text x="56.1" y="1.35" size="0.635" layer="21" font="vector" ratio="20">GND</text>
+<wire x1="55.7" y1="2.7" x2="55.7" y2="2.4" width="0.2" layer="21"/>
+<wire x1="55.7" y1="2.4" x2="58.3" y2="2.4" width="0.2" layer="21"/>
+<wire x1="58.3" y1="2.4" x2="58.3" y2="2.7" width="0.2" layer="21"/>
+<wire x1="60.8" y1="2.7" x2="60.8" y2="2.4" width="0.2" layer="21"/>
+<wire x1="60.8" y1="2.4" x2="63.4" y2="2.4" width="0.2" layer="21"/>
+<wire x1="63.4" y1="2.4" x2="63.4" y2="2.7" width="0.2" layer="21"/>
 </plain>
 <attributes>
@@
 <attribute name="VALUE" x="57.18" y="28.17" size="0.4064" layer="27" font="vector" ratio="15" rot="R270"/>
 </element>
-<element name="C17" library="oresat-rcl" package=".0805-C-NOSILK" value="22u" x="43.96" y="36.27" smashed="yes">
+<element name="C17" library="oresat-rcl" package=".0805-C-NOSILK" value="22uF" x="43.96" y="36.27" smashed="yes">
 <attribute name="NAME" x="42.96" y="37.02" size="0.4064" layer="25" font="vector" ratio="15"/>
 <attribute name="NAME" x="43.96" y="36.27" size="0.3" layer="33" ratio="15" align="center"/>
@@
 <attribute name="VALUE" x="73.495" y="6.525" size="0.4064" layer="27"/>
 </element>
-<element name="R13" library="oresat-rcl" package=".0603-C-NOSILK" value="1.7K" x="68.35" y="8.11" smashed="yes" rot="R90">
+<element name="R13" library="oresat-rcl" package=".0603-C-NOSILK" value="1.69K" x="68.35" y="8.11" smashed="yes" rot="R90">
 <attribute name="NAME" x="69.315" y="7.575" size="0.4064" layer="25" rot="R90"/>
 <attribute name="VALUE" x="70.255" y="7.475" size="0.4064" layer="27" rot="R90"/>
@@
 <attribute name="VALUE" x="78.035" y="34.555" size="0.4064" layer="27" rot="R180"/>
 </element>
-<element name="R15" library="oresat-rcl" package=".0603-C-NOSILK" value="26.36K" x="88.79" y="45.13" smashed="yes" rot="R180">
+<element name="R15" library="oresat-rcl" package=".0603-C-NOSILK" value="26.4K" x="88.79" y="45.13" smashed="yes" rot="R180">
 <attribute name="DIS" value="Digi-Key" x="54.5" y="109.9" size="1.778" layer="27" rot="R180" display="off"/>
 <attribute name="DPN" value="1276-4275-1-ND" x="54.5" y="109.9" size="1.778" layer="27" rot="R180" display="off"/>
@@
 <attribute name="VALUE" x="44.96" y="35.28" size="0.4064" layer="27" font="vector" ratio="15" rot="R180"/>
 </element>
-<element name="R26" library="oresat-rcl" package=".0603-C-NOSILK" value="50" x="26.25" y="5.97" smashed="yes" rot="R270">
+<element name="R26" library="oresat-rcl" package=".0603-C-NOSILK" value="51.1" x="26.25" y="5.97" smashed="yes" rot="R270">
 <attribute name="NAME" x="26.885" y="6.405" size="0.4064" layer="25" rot="R270"/>
 <attribute name="VALUE" x="24.345" y="6.605" size="0.4064" layer="27" rot="R270"/>
 </element>
-<element name="R27" library="oresat-rcl" package=".0603-C-NOSILK" value="50" x="28.03" y="5.97" smashed="yes" rot="R270">
+<element name="R27" library="oresat-rcl" package=".0603-C-NOSILK" value="51.1" x="28.03" y="5.97" smashed="yes" rot="R270">
 <attribute name="NAME" x="28.665" y="6.405" size="0.4064" layer="25" rot="R270"/>
 <attribute name="VALUE" x="26.125" y="6.605" size="0.4064" layer="27" rot="R270"/>
 </element>
-<element name="R28" library="oresat-rcl" package=".0603-C-NOSILK" value="50" x="44.77" y="14.33" smashed="yes">
+<element name="R28" library="oresat-rcl" package=".0603-C-NOSILK" value="10K" x="44.77" y="14.33" smashed="yes">
 <attribute name="NAME" x="44.335" y="13.265" size="0.4064" layer="25"/>
 <attribute name="VALUE" x="44.135" y="12.425" size="0.4064" layer="27"/>
@@
 <attribute name="VALUE" x="13.405" y="45.875" size="0.4064" layer="27" rot="R180"/>
 </element>
-<element name="R8" library="oresat-rcl" package=".0603-C-NOSILK" value="439" x="13.27" y="40.61" smashed="yes">
+<element name="R8" library="oresat-rcl" package=".0603-C-NOSILK" value="442" x="13.27" y="40.61" smashed="yes">
 <attribute name="NAME" x="13.135" y="39.545" size="0.4064" layer="25"/>
 <attribute name="VALUE" x="12.635" y="38.705" size="0.4064" layer="27"/>
 </element>
-<element name="R9" library="oresat-rcl" package=".0603-C-NOSILK" value="439" x="106.67" y="48.39" smashed="yes" rot="R180">
+<element name="R9" library="oresat-rcl" package=".0603-C-NOSILK" value="442" x="106.67" y="48.39" smashed="yes" rot="R180">
 <attribute name="NAME" x="106.805" y="47.755" size="0.4064" layer="25" rot="R180"/>
 <attribute name="VALUE" x="107.305" y="50.295" size="0.4064" layer="27" rot="R180"/>
@@
 </element>
 <element name="JP3" library="pinhead" library_urn="urn:adsk.eagle:library:325" package="1X03" package3d_urn="urn:adsk.eagle:package:22458/2" value="" x="79.4" y="18.5" smashed="yes">
-<attribute name="NAME" x="78.3138" y="15.8288" size="0.8128" layer="25" font="vector" ratio="10"/>
 <attribute name="POPULARITY" value="92" x="79.4" y="18.5" size="1.778" layer="27" display="off"/>
 <attribute name="VALUE" x="75.59" y="15.325" size="1.27" layer="27"/>
@@
 <via x="102.3" y="11.4" extent="1-16" drill="0.35"/>
 <via x="94.5" y="19.2" extent="1-16" drill="0.35"/>
-<via x="89.4" y="25.8" extent="1-16" drill="0.35"/>
+<via x="90.5" y="24.4" extent="1-16" drill="0.35"/>
 <via x="92.3" y="25.9" extent="1-16" drill="0.35"/>
 <via x="87.4" y="41.1" extent="1-16" drill="0.35"/>
@@
 <wire x1="78.2" y1="11.9" x2="78.8" y2="11.9" width="0.5" layer="1"/>
 <wire x1="78.2" y1="10.1024" x2="78.2" y2="11.9" width="0.5" layer="1"/>
-<wire x1="76.9" y1="12.4674" x2="76.9" y2="12.5" width="0.5" layer="1"/>
 <contactref element="IC1" pad="3"/>
 <wire x1="86.265" y1="11.235" x2="86.265" y2="9.612" width="0.5" layer="1"/>
@@
 <wire x1="37.73" y1="32.54" x2="40.77" y2="32.54" width="0.2" layer="1"/>
 <wire x1="40.77" y1="32.54" x2="41.46" y2="32.54" width="0.2" layer="1"/>
-<wire x1="50" y1="24" x2="50" y2="22.1" width="0.2" layer="1"/>
-<via x="50" y="22.1" extent="1-16" drill="0.35"/>
-<wire x1="50" y1="22.1" x2="51.7" y2="20.4" width="0.2" layer="16"/>
-<wire x1="51.7" y1="20.4" x2="51.7" y2="16.2" width="0.2" layer="16"/>
+<wire x1="50" y1="24" x2="50" y2="22.5" width="0.2" layer="1"/>
+<via x="50" y="22.5" extent="1-16" drill="0.35"/>
+<wire x1="50" y1="22.5" x2="51.7" y2="20.8" width="0.2" layer="16"/>
+<wire x1="51.7" y1="20.8" x2="51.7" y2="16.2" width="0.2" layer="16"/>
 <via x="51.7" y="16.2" extent="1-16" drill="0.35"/>
 <wire x1="51.7" y1="16.2" x2="54.3" y2="13.6" width="0.2" layer="1"/>
@@
 <wire x1="99.11" y1="32.71" x2="99" y2="32.6" width="0.2" layer="1"/>
 <via x="99" y="32.6" extent="1-16" drill="0.35"/>
-<wire x1="84.715" y1="1.915" x2="84.7" y2="1.9" width="0.2" layer="1"/>
 <via x="84.7" y="1.9" extent="1-16" drill="0.35"/>
 <wire x1="84.7" y1="1.9" x2="99" y2="16.2" width="0.2" layer="16"/>
@@
 <contactref element="U1" pad="19"/>
 <contactref element="R33" pad="1"/>
-<wire x1="85.985" y1="1.915" x2="86" y2="1.9" width="0.2" layer="1"/>
 <via x="86" y="1.9" extent="1-16" drill="0.35"/>
 <wire x1="96.26" y1="34.48" x2="94.42" y2="34.48" width="0.2" layer="1"/>
@@
 <signal name="N$2">
 <contactref element="R8" pad="1"/>
-<wire x1="12.56" y1="40.62" x2="12.57" y2="40.61" width="0.2" layer="1"/>
 <contactref element="Q4" pad="CAT"/>
 <wire x1="12.57" y1="40.61" x2="9.76" y2="40.61" width="0.2" layer="1"/>
@@
 <signal name="N$5">
 <contactref element="R9" pad="1"/>
-<wire x1="107.37" y1="48.39" x2="107.48" y2="48.28" width="0.2" layer="1"/>
 <contactref element="Q5" pad="CAT"/>
 <wire x1="107.37" y1="48.39" x2="111.044" y2="48.39" width="0.2" layer="1"/>
@@
 <contactref element="R22" pad="2"/>
 <contactref element="U$5" pad="CSP"/>
-<wire x1="60.29" y1="28.27" x2="60.29" y2="28.81" width="0.2" layer="1"/>
 <wire x1="65.7" y1="32.98" x2="65.7" y2="30.18" width="1" layer="1"/>
 <wire x1="65.7" y1="30.18" x2="63.79" y2="28.27" width="1" layer="1"/>
@@
 </signal>
 <signal name="GND3">
-<via x="89.4" y="22.1" extent="1-16" drill="0.35"/>
+<via x="90.5" y="22" extent="1-16" drill="0.35"/>
 </signal>
 <signal name="GND4">
@@
 </signal>
 <signal name="GND12">
-<via x="55.6" y="1.6" extent="1-16" drill="0.35"/>
+<via x="55" y="1.8" extent="1-16" drill="0.35"/>
 </signal>
 <signal name="GND13">
-<via x="58.2" y="1.6" extent="1-16" drill="0.35"/>
+<via x="58.8" y="1.7" extent="1-16" drill="0.35"/>
 </signal>
 <signal name="GND14">
@@
 <mfgpreviewcolor name="substratecolor" color="0xFF786E46"/>
 </mfgpreviewcolors>
+<errors>
+</errors>
 </board>
 </drawing>

Commit message: completed BOM except for a couple pin head connectors
Parts:
- removed IC1: BD62120AEFJ-E2, SamacSys_Parts:SOIC127P600X100-9N
- removed R6: NP, oresat-rcl:.0603-C-NOSILK
- added U2: BD62120AEFJ-E2, SamacSys_Parts:SOIC127P600X100-9N
- C13: value 0.1u -> 100n
- L1: value 1.5 uH -> 1.5uH; device L-Coilcraft-XFL4020:L-COILCRAFT-XFL4020 -> L--IHLP2020CZER1R5M11--1.5uHInductor:IHLP2020CZER1R5M11
- L2: value L-COILCRAFT-XFL4020 -> 4.7uH; device L-Coilcraft-XFL4020:L-COILCRAFT-XFL4020 -> L--IHLP2020BZER4R7M11--4.7uInductor:IHLP2020BZER4R7M11
- R10, R16, R28, R32, R33, R34, R35, R36, R7: value 10K -> 10k
- R11, R12: value 1K -> 1k
- R13: value 1.69K -> 1.69k
- R14: value 3.3K -> 3.3k
- R15: value 26.4K -> 26.4k
- R17: value (none) -> 10k
- R20: value (none) -> 2.4k
- R3: value 150K -> 150k
- R5: value NP -> 100k
- moved L1 4.08 mm to (27.4, 30.3)
- moved D2 3.31 mm to (73.3, 33.6)
- moved L2 2.10 mm to (67.5, 33.1)
Connections:
- new net N$3: U2.7
- net +12V: now also U2.3; no longer IC1.3
- net GND: now also U2.1, U2.4, U2.9; no longer IC1.1, IC1.4, IC1.7, IC1.9, R6.1
- net IN1: now also U2.5; no longer IC1.5
- net IN2: now also U2.6; no longer IC1.6
- net LAMOTOR+: now also U2.2; no longer IC1.2
- net LAMOTOR-: now also U2.8; no longer IC1.8
- net N$10: now also L2.P$1; no longer L2.1
- net N$28: now also L2.P$2; no longer L2.2
- net TPS-EN: no longer R6.2
- net TPS-L1: now also L1.P$1; no longer L1.1
- net TPS-L2: now also L1.P$2; no longer L1.2
Routing:
- net GND: track 16.0 -> 8.96 mm
- net TPS-L2: track 4.91 -> 10.1 mm
- net TPS-L1: track 3.58 -> 7.25 mm
- net N$10: track 10.0 -> 13.4 mm
- net TPS-EN: track 10.1 -> 8.51 mm
